File: board/pcc_circuit_example.brd (EAGLE design)
At the start: 52 x 29.1 mm, 18 parts, among them T1 BT138-V

Commit message: little improvements
Parts:
- moved B1 0.38 mm to (17.3, 24.0)
Other:
- board text added: "Phase- CutCtrl github.com/ benoitjoh"
- board text removed: "Phase- CutCtrl (c) jbenoit 2018"
Changed lines of the file:
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@@
 <layer number="20" name="Dimension" color="15" fill="1" visible="yes" active="yes"/>
 <layer number="21" name="tPlace" color="7" fill="1" visible="yes" active="yes"/>
-<layer number="22" name="bPlace" color="7" fill="1" visible="no" active="yes"/>
+<layer number="22" name="bPlace" color="7" fill="1" visible="yes" active="yes"/>
 <layer number="23" name="tOrigins" color="15" fill="1" visible="yes" active="yes"/>
-<layer number="24" name="bOrigins" color="15" fill="1" visible="no" active="yes"/>
+<layer number="24" name="bOrigins" color="15" fill="1" visible="yes" active="yes"/>
 <layer number="25" name="tNames" color="7" fill="1" visible="no" active="yes"/>
 <layer number="26" name="bNames" color="7" fill="1" visible="no" active="yes"/>
 <layer number="27" name="tValues" color="7" fill="1" visible="yes" active="yes"/>
 <layer number="28" name="bValues" color="7" fill="1" visible="yes" active="yes"/>
-<layer number="29" name="tStop" color="7" fill="3" visible="yes" active="yes"/>
-<layer number="30" name="bStop" color="7" fill="6" visible="no" active="yes"/>
+<layer number="29" name="tStop" color="7" fill="3" visible="no" active="yes"/>
+<layer number="30" name="bStop" color="7" fill="6" visible="yes" active="yes"/>
 <layer number="31" name="tCream" color="7" fill="4" visible="no" active="yes"/>
 <layer number="32" name="bCream" color="7" fill="5" visible="no" active="yes"/>
@@
 <layer number="37" name="tTest" color="7" fill="1" visible="no" active="yes"/>
 <layer number="38" name="bTest" color="7" fill="1" visible="no" active="yes"/>
-<layer number="39" name="tKeepout" color="4" fill="11" visible="yes" active="yes"/>
-<layer number="40" name="bKeepout" color="1" fill="11" visible="no" active="yes"/>
+<layer number="39" name="tKeepout" color="4" fill="11" visible="no" active="yes"/>
+<layer number="40" name="bKeepout" color="1" fill="11" visible="yes" active="yes"/>
 <layer number="41" name="tRestrict" color="4" fill="10" visible="no" active="yes"/>
 <layer number="42" name="bRestrict" color="1" fill="10" visible="no" active="yes"/>
@@
 <wire x1="22.352" y1="6.985" x2="18.796" y2="8.509" width="0.4064" layer="27"/>
 <wire x1="20.447" y1="8.509" x2="21.59" y2="8.509" width="0.4064" layer="27"/>
-<text x="31.496" y="6.985" size="1.27" layer="28" font="vector" rot="MR0">for resistive load:
+<text x="30.353" y="8.255" size="1.27" layer="28" font="vector" rot="MR0">for resistive load:
 no C1, R1=0</text>
 <text x="10.033" y="13.462" size="1.27" layer="28" font="vector" ratio="10" rot="MR90">AC in</text>
@@
 <wire x1="9.525" y1="9.652" x2="9.525" y2="1.778" width="0.4064" layer="28"/>
 <wire x1="9.525" y1="1.778" x2="10.541" y2="1.778" width="0.4064" layer="28"/>
-<text x="18.034" y="17.399" size="1.27" layer="27" font="vector" ratio="10" rot="R180">R1</text>
+<text x="17.907" y="17.526" size="1.27" layer="27" font="vector" ratio="10" rot="R180">R1</text>
 <text x="29.845" y="10.541" size="1.27" layer="27" font="vector" ratio="10" rot="R180">C1</text>
-<text x="36.449" y="10.922" size="1.016" layer="16" font="vector" ratio="10" rot="MR270">Phase-
+<text x="36.195" y="11.43" size="1.016" layer="16" font="vector" ratio="10" rot="MR270">Phase-
 CutCtrl
-(c) jbenoit
-2018</text>
+github.com/
+benoitjoh
+</text>
 </plain>
 <attributes>
@@
 </autorouter>
 <elements>
-<element name="B1" library="rectifier" package="RB1A" value="201G" x="17.653" y="24.003" rot="R90"/>
+<element name="B1" library="rectifier" package="RB1A" value="201G" x="17.272" y="24.003" rot="R90"/>
 <element name="C3" library="capacitor-wima" package="C15B5" value="100n" x="22.225" y="13.335"/>
 <element name="C7" library="bauteile_jbt" package="C050-024X044" value="100n" x="46.99" y="17.526" rot="R270"/>
@@
 </element>
 <element name="Q4" library="bauteile_jbt" package="TO92-EBC" value="" x="42.545" y="20.32" rot="R180"/>
-<element name="R14" library="bauteile_jbt" package="R_0207/2V" value="47k" x="24.384" y="20.193" rot="R270"/>
-<element name="R2" library="bauteile_jbt" package="R_0207/2V" value="10k" x="46.482" y="24.638" rot="R180"/>
-<element name="R4" library="bauteile_jbt" package="R_0207/2V" value="47k" x="25.019" y="25.4" rot="R270"/>
-<element name="R6" library="bauteile_jbt" package="R_0207/2V" value="120" x="28.194" y="17.399" rot="R180"/>
-<element name="R7" library="bauteile_jbt" package="R_0207/2V" value="1.2k" x="19.685" y="17.526" rot="R180"/>
+<element name="R14" library="bauteile_jbt" package="R_0207/2V" value="47k" x="24.384" y="20.193" smashed="yes" rot="R270">
+<attribute name="NAME" x="25.4" y="20.2438" size="1.016" layer="25" font="vector" ratio="10" rot="R270"/>
+<attribute name="VALUE" x="22.3266" y="20.5232" size="1.27" layer="27" font="vector" ratio="10" rot="R270"/>
+</element>
+<element name="R2" library="bauteile_jbt" package="R_0207/2V" value="10k" x="46.482" y="24.638" smashed="yes" rot="R180">
+<attribute name="NAME" x="46.5328" y="23.622" size="1.016" layer="25" font="vector" ratio="10" rot="R180"/>
+<attribute name="VALUE" x="48.3362" y="27.4574" size="1.27" layer="27" font="vector" ratio="10" rot="R180"/>
+</element>
+<element name="R4" library="bauteile_jbt" package="R_0207/2V" value="47k" x="25.019" y="25.4" smashed="yes" rot="R270">
+<attribute name="NAME" x="26.035" y="25.4508" size="1.016" layer="25" font="vector" ratio="10" rot="R270"/>
+<attribute name="VALUE" x="22.7076" y="26.1112" size="1.27" layer="27" font="vector" ratio="10" rot="R270"/>
+</element>
+<element name="R6" library="bauteile_jbt" package="R_0207/2V" value="120" x="28.194" y="17.399" smashed="yes" rot="R180">
+<attribute name="NAME" x="28.2448" y="16.383" size="1.016" layer="25" font="vector" ratio="10" rot="R180"/>
+<attribute name="VALUE" x="29.2862" y="20.0914" size="1.27" layer="27" font="vector" ratio="10" rot="R180"/>
+</element>
+<element name="R7" library="bauteile_jbt" package="R_0207/2V" value="1.2k" x="19.685" y="17.526" smashed="yes" rot="R180">
+<attribute name="NAME" x="19.7358" y="16.51" size="1.016" layer="25" font="vector" ratio="10" rot="R180"/>
+<attribute name="VALUE" x="19.8882" y="19.7104" size="1.27" layer="27" font="vector" ratio="10" rot="R180"/>
+</element>
 <element name="R8" library="bauteile_jbt" package="R_0207/2V" value="330" x="46.355" y="12.446"/>
-<element name="R9" library="bauteile_jbt" package="R_0207/2V" value="10k" x="41.148" y="26.543"/>
+<element name="R9" library="bauteile_jbt" package="R_0207/2V" value="10k" x="41.148" y="26.543" smashed="yes">
+<attribute name="NAME" x="41.0972" y="27.559" size="1.016" layer="25" font="vector" ratio="10"/>
+<attribute name="VALUE" x="40.1828" y="23.8506" size="1.27" layer="27" font="vector" ratio="10"/>
+</element>
 <element name="T1" library="bauteile_jbt" package="TO220V" value="BT138-V" x="23.622" y="1.905" rot="R180"/>
 <element name="X1" library="bauteile_jbt" package="AK300/4" value="" x="6.223" y="10.795" rot="R90">
@@
 <wire x1="4.318" y1="19.812" x2="5.715" y2="21.209" width="0.4064" layer="16"/>
 <wire x1="5.715" y1="21.209" x2="9.779" y2="21.209" width="0.4064" layer="16"/>
-<wire x1="9.779" y1="21.209" x2="15.113" y2="26.543" width="0.4064" layer="16"/>
+<wire x1="9.779" y1="21.209" x2="14.732" y2="26.543" width="0.4064" layer="16"/>
 <wire x1="23.622" y1="4.445" x2="23.622" y2="7.239" width="2.54" layer="1"/>
 <wire x1="23.622" y1="7.239" x2="22.098" y2="8.763" width="2.54" layer="1"/>
@@
 <wire x1="9.144" y1="8.255" x2="7.1374" y2="8.255" width="2.54" layer="16"/>
 <wire x1="7.1374" y1="8.255" x2="6.223" y2="8.2804" width="1.524" layer="16"/>
-<wire x1="20.193" y1="21.463" x2="18.288" y2="21.463" width="0.4064" layer="16"/>
+<wire x1="19.812" y1="21.463" x2="18.288" y2="21.463" width="0.4064" layer="16"/>
 <wire x1="18.288" y1="21.463" x2="16.002" y2="19.177" width="0.4064" layer="16"/>
 <wire x1="16.002" y1="19.177" x2="8.001" y2="19.177" width="0.4064" layer="16"/>
@@
 <contactref element="R14" pad="2"/>
 <contactref element="B1" pad="-"/>
-<wire x1="20.193" y1="26.543" x2="20.193" y2="23.622" width="0.4064" layer="16"/>
-<wire x1="20.193" y1="23.622" x2="21.844" y2="21.971" width="0.4064" layer="16"/>
+<wire x1="19.812" y1="26.543" x2="19.812" y2="24.003" width="0.4064" layer="16"/>
+<wire x1="19.812" y1="24.003" x2="21.844" y2="21.971" width="0.4064" layer="16"/>
 <wire x1="21.844" y1="21.971" x2="21.844" y2="20.066" width="0.4064" layer="16"/>
 <wire x1="21.844" y1="20.066" x2="22.987" y2="18.923" width="0.4064" layer="16"/>
@@
 <contactref element="R4" pad="2"/>
 <contactref element="B1" pad="+"/>
-<wire x1="15.113" y1="21.463" x2="15.113" y2="24.003" width="0.4064" layer="16"/>
-<wire x1="15.113" y1="24.003" x2="19.558" y2="27.94" width="0.4064" layer="16"/>
-<wire x1="19.558" y1="27.94" x2="21.59" y2="27.94" width="0.4064" layer="16"/>
+<wire x1="14.732" y1="21.463" x2="14.732" y2="23.876" width="0.4064" layer="16"/>
+<wire x1="14.732" y1="23.876" x2="19.304" y2="27.94" width="0.4064" layer="16"/>
+<wire x1="19.304" y1="27.94" x2="21.59" y2="27.94" width="0.4064" layer="16"/>
 <wire x1="21.59" y1="27.94" x2="22.352" y2="27.178" width="0.4064" layer="16"/>
 <wire x1="22.352" y1="27.178" x2="22.352" y2="24.892" width="0.4064" layer="16"/>
